File: subsheet_03.kicad_sch (KiCad schematic)
At the start: 0 parts

Commit message: Start MFP, with builtin RSVE mod
Parts:
- added C401: 0.22uF, symbol Device:C_Small
- added C402, C403: 30pF, symbol Device:C_Small
- added J401: RSVE LED, symbol Connector_Generic:Conn_01x02
- added JP401: NO RSVE, symbol Jumper:SolderJumper_2_Open
- added R401: 1K, symbol Device:R_Small_US
- added R402, R403: 2K2, symbol Device:R_Small_US
- added SW401: SW_Push, symbol Switch:SW_Push
- added U401: 74HC4040 12 stage counter, Package_DIP:DIP-16_W7.62mm_LongPads, symbol 74x4040:12-STAGE_BINARY_RIPPLE_COUNTER_PHY
- added U402: GAL16V8, Package_DIP:DIP-20_W7.62mm_LongPads, symbol gal16v8:HIGH_PERFORMANCE_E2_CMOS_PLD_GENERIC_ARRAY_LOGIC_PHY
- added U403: MC68901_MULTI_FUNCTION_PERIPHERAL_PLCC_52_PHY, Package_LCC:PLCC-52_THT-Socket, symbol mc68901d-plcc52:MC68901_MULTI_FUNCTION_PERIPHERAL_PLCC_52_PHY
- added X401: 1.8432 MHz, Oscillator:Oscillator_DIP-8, symbol Oscillator:CXO_DIP8
- added Y401: 2.4576 MHz, symbol Device:Crystal_Small
Connections:
- new net: C402.1, U403.19 (XTAL1), Y401.1
- new net: C403.1, U403.20 (XTAL2), Y401.2
- new net: R403.1, U403.28 (I3)
- new net: R402.1, SW401.1, U403.32 (I7)
- new net: U401.13 (Q7), U402.8 (I)
- new net: U401.2 (Q5), U402.4 (I)
- new net: U401.3 (Q4), U402.5 (I)
- new net: U401.4 (Q6), U402.6 (I)
- new net: U401.5 (Q3), U402.7 (I)
- new net A1: U403.3 (RS1)
- new net A2: U403.4 (RS2)
- new net A3: U403.5 (RS3)
- new net A4: U403.6 (RS4)
- new net A5: U403.7 (RS5)
- new net CPLD_MFP_ACIA_IRQ: U403.29 (I4)
- new net CPLD_MFP_MEDIA_IRQ: U403.30 (I5)
- new net CPU_R/~{W}: U403.2 (R/~{W})
- new net D0: U403.41 (D0)
- new net D1: U403.42 (D1)
- new net D2: U403.43 (D2)
- new net D3: U403.44 (D3)
- new net D4: U403.45 (D4)
- new net D5: U403.46 (D5)
- new net D6: U403.47 (D6)
- new net D7: U403.48 (D7)
- new net GND: C401.2, C402.2, C403.2, SW401.2, U401.8 (GND), U402.10 (GND), U402.11 (I/~{OE}), U403.38 (~{IEI}), U403.40 (GND), X401.4 (GND)
- new net MFP_CLOCK: U403.39 (CLK)
- new net MFP_SERIAL_CLOCK: JP401.2 (B), U402.14 (I/O/Q), U403.11 (RC), U403.8 (TC)
- new net MFP_Serial_IN: U403.10 (SI)
- new net MFP_Serial_OUT: U403.9 (SO)
- new net MFP_TDO: JP401.1 (A), U402.2 (I), U403.18 (TDO)
- new net RSVE_CLK: U402.1 (I/CLK), U402.9 (I), X401.5 (OUT)
- new net RSVE_CP: U401.10 (~{CP}), U402.13 (I/O/Q)
- new net RSVE_MR: U401.11 (MR), U402.12 (I/O/Q)
- new net VCC: C401.1, R401.1, R402.2, R403.2, U401.16 (VCC), U402.3 (I), U403.12 (VCC), X401.8 (Vcc)
- new net led+: J401.1 (Pin_1), R401.2
- new net led-: J401.2 (Pin_2), U402.15 (I/O/Q)
- new net ~{CPLD_MFP_CS}: U403.52 (~{CS})
- new net ~{CPLD_MFP_IACK}: U403.49 (~{IACK})
- new net ~{CPLD_MFP_IRQ}: U403.36 (~{IRQ})
- new net ~{CPU_DTACK}: U403.50 (~{DTACK})
- new net ~{CPU_LDS}: U403.51 (~{DS})
- new net ~{CPU_RESET}: U403.24 (~{RESET})
- no-connect marks 0 -> 18
Other:
- note added: "BUILTIN RSVE MOD"
- note added: "Closed only if RSVE MOD is not populated."
- note added: "DEPRECATED, for use with a regular TOS or EMUTOS that relies on it. Switch to select either color display (open) or monochrome display (closed)."
- note added: "See https://github.com/sporniket/atari-st-mod-serial-port-upgrade-rsve"
- note added: "TODO : Serial port * All in one IC with a single power rail to support RS-232 * A header pin connector for a CH340E <--> micro USB-B breakout"
- note added: "TODO : emit DE from FPGA ?"
- note added: "TODO : linked to serial port"
- note added: "TODO : parallel busy is active high or low ??"
- note added: "TODO linked to serial port"
