File: subsheet_07.kicad_sch (KiCad schematic)
At the start: 0 parts

Commit message: Started FPGA module
Parts:
- added J801: P2, Connector_PinHeader_2.54mm:PinHeader_2x15_P2.54mm_Vertical, symbol colorlight_i9_v7.2_p2:COLORLIGHT_I9_V7.2_EXPANSION_CONNECTOR_P2_PHY
- added J802: P3, Connector_PinHeader_2.54mm:PinHeader_2x15_P2.54mm_Vertical, symbol colorlight_i9_v7.2_p3:COLORLIGHT_I9_V7.2_EXPANSION_CONNECTOR_P3_PHY
- added J803: P4, Connector_PinHeader_2.54mm:PinHeader_2x15_P2.54mm_Vertical, symbol colorlight_i9_v7.2_p4:COLORLIGHT_I9_V7.2_EXPANSION_CONNECTOR_P4_PHY
- added J804: P5, Connector_PinHeader_2.54mm:PinHeader_2x15_P2.54mm_Vertical, symbol colorlight_i9_v7.2_p5:COLORLIGHT_I9_V7.2_EXPANSION_CONNECTOR_P5_PHY
- added J805: P6, Connector_PinHeader_2.54mm:PinHeader_2x15_P2.54mm_Vertical, symbol colorlight_i9_v7.2_p6:COLORLIGHT_I9_V7.2_EXPANSION_CONNECTOR_P6_PHY
- added NT801: NetTie_2, symbol Device:NetTie_2
Connections:
- new net +3V3: NT801.1
- new net 3V3_FPGA: J801.1 (3V3), J801.19 (3V3), J801.2 (3V3), J801.20 (3V3), J802.1 (3V3), J802.19 (3V3), J802.2 (3V3), J802.20 (3V3), J803.1 (3V3), J803.19 (3V3), J803.2 (3V3), J803.20 (3V3), J804.1 (3V3), J804.19 (3V3), J804.2 (3V3), J804.20 (3V3), J805.1 (3V3), J805.19 (3V3), J805.2 (3V3), J805.20 (3V3), NT801.2
- new net A0: J805.30 (R1)
- new net A1: J805.29 (T1)
- new net A10: J805.10 (M4)
- new net A11: J805.9 (L4)
- new net A12: J805.8 (L5)
- new net A13: J805.7 (P16)
- new net A14: J805.6 (J16)
- new net A15: J805.5 (J18)
- new net A16: J804.12 (D18)
- new net A17: J804.11 (D17)
- new net A18: J804.10 (G5)
- new net A19: J804.9 (D16)
- new net A2: J805.28 (U1)
- new net A20: J804.8 (F5)
- new net A21: J804.7 (E6)
- new net A22: J804.6 (E5)
- new net A23: J804.5 (F4)
- new net A3: J805.27 (Y2)
- new net A4: J805.26 (W1)
- new net A5: J805.25 (V1)
- new net A6: J805.24 (M1)
- new net A7: J805.23 (N2)
- new net A8: J805.12 (R3)
- new net A9: J805.11 (N4)
- new net CDPL_FPGA_CS: J804.13 (E17)
- new net CPU_R/~{W}: J804.23 (E18)
- new net D0: J801.30 (J20)
- new net D1: J801.29 (G20)
- new net D10: J801.10 (R18)
- new net D11: J801.9 (R17)
- new net D12: J801.8 (C18)
- new net D13: J801.7 (T18)
- new net D14: J801.6 (L2)
- new net D15: J801.5 (K18)
- new net D16: J802.30 (D1)
- new net D17: J802.29 (E2)
- new net D18: J802.28 (C1)
- new net D19: J802.27 (D2)
- new net D2: J801.28 (L18)
- new net D20: J802.26 (C2)
- new net D21: J802.25 (B1)
- new net D22: J802.24 (E3)
- new net D23: J802.23 (A3)
- new net D24: J802.12 (C17)
- new net D25: J802.11 (A18)
- new net D26: J802.10 (B18)
- new net D27: J802.9 (A19)
- new net D28: J802.8 (B20)
- new net D29: J802.7 (B19)
- new net D3: J801.27 (K20)
- new net D30: J802.6 (F20)
- new net D31: J802.5 (D20)
- new net D4: J801.26 (M18)
- new net D5: J801.25 (L20)
- new net D6: J801.24 (N17)
- new net D7: J801.23 (N18)
- new net D8: J801.12 (P17)
- new net D9: J801.11 (M17)
- new net GND: J801.15 (GND), J801.21 (GND), J801.22 (GND), J801.3 (GND), J801.4 (GND), J802.15 (GND), J802.21 (GND), J802.22 (GND), J802.3 (GND), J802.4 (GND), J803.15 (GND), J803.21 (GND), J803.22 (GND), J803.3 (GND), J803.4 (GND), J804.15 (GND), J804.21 (GND), J804.22 (GND), J804.3 (GND), J804.4 (GND), J805.15 (GND), J805.21 (GND), J805.3 (GND)
- new net ~{CPU_AS}: J805.13 (T3)
- new net ~{CPU_DTACK}: J804.24 (G16)
- new net ~{CPU_LDS}: J804.18 (F17)
- new net ~{CPU_UDS}: J804.17 (F16)
- no-connect marks 0 -> 11
Other:
- note added: "TODO : a circuit to select power source and protect the FPGA module"
